Commit message: drl-v0

File: rotors_description/urdf/component_snippets.xacro (robot description, xacro)
@@ -682,7 +682,7 @@
       </visual>
       <inertial>
-        <mass value="0.13" />
-        <origin xyz="0 0 0" rpy="0 0 0" />
-        <inertia ixx="1e-6" ixy="0" ixz="0" iyy="1e-6" iyz="0" izz="1e-6" />
+        <mass value="0.00" />
+        <origin xyz="0 0 0" rpy="0 0 0" />
+        <inertia ixx="0e-6" ixy="0" ixz="0" iyy="0e-6" iyz="0" izz="0e-6" />
       </inertial>
     </link>
@@ -710,6 +710,8 @@
     </xacro:if>
     <!-- Groundtruth -->
-    <xacro:if value="${enable_ground_truth}">
+    <!--
+    <xacro:if value="${enable_ground_truth}"> -->
       <!-- Odometry Sensor -->
+      <!--
       <xacro:odometry_plugin_macro
         namespace="${namespace}/ground_truth"
@@ -738,9 +740,11 @@
         odometry_map=""
         image_scale="">
-        <inertia ixx="0.00001" ixy="0.0" ixz="0.0" iyy="0.00001" iyz="0.0" izz="0.00001" /> <!-- [kg m^2] [kg m^2] [kg m^2] [kg m^2] [kg m^2] [kg m^2] -->
-        <origin xyz="0.0 0.0 0.0" rpy="0.0 0.0 0.0" />
+        <inertia ixx="0.00001" ixy="0.0" ixz="0.0" iyy="0.00001" iyz="0.0" izz="0.00001" />  --> <!-- [kg m^2] [kg m^2] [kg m^2] [kg m^2] [kg m^2] [kg m^2] -->
+      <!--
+      <origin xyz="0.0 0.0 0.0" rpy="0.0 0.0 0.0" />
       </xacro:odometry_plugin_macro>
-    </xacro:if>
+    </xacro:if>  -->
     <!-- ADIS16448 IMU. -->
+    <!--
     <xacro:imu_plugin_macro
       namespace="${namespace}"
@@ -759,5 +763,5 @@
       <inertia ixx="0.00001" ixy="0.0" ixz="0.0" iyy="0.00001" iyz="0.0" izz="0.00001" />
       <origin xyz="0.015 0 0.0113" rpy="0 0 0" />
-    </xacro:imu_plugin_macro>
+    </xacro:imu_plugin_macro>  -->
   </xacro:macro>
   <xacro:macro name="ground_truth_imu_and_odometry" params="namespace parent_link">
